File: KiCad project/FPGA_Peripherals.sch (KiCad schematic (older format))
At the start: 36 parts, among them IC1 ADS7924IRTER, IC2 NCP114BSN330T1G, J5 L77HDE15SD1CH4RHNVGA

Commit message: Update
Parts:
- C3, C4, C6: symbol TFG20:C100n -> TFG20-rescue:C100n-TFG20-TFG20-rescue
- C5: symbol TFG20:C10u -> TFG20-rescue:C10u-TFG20-TFG20-rescue
- FB1, FB2: symbol TFG20:BLM18KG331SN1D -> TFG20-rescue:BLM18KG331SN1D-TFG20-TFG20-rescue
- IC1: symbol TFG20:ADS7924IRTER -> TFG20-rescue:ADS7924IRTER-TFG20-TFG20-rescue
- IC2: symbol TFG20:NCP114BSN330T1G -> TFG20-rescue:NCP114BSN330T1G-TFG20-TFG20-rescue
- J5: symbol TFG20:L77HDE15SD1CH4RHNVGA -> TFG20-rescue:L77HDE15SD1CH4RHNVGA-TFG20-TFG20-rescue
- R10, R9: symbol TFG20:R10k -> TFG20-rescue:R10k-TFG20-TFG20-rescue
- R11, R12, R13, R14, R21, R34, R35: symbol TFG20:R100 -> TFG20-rescue:R100-TFG20-TFG20-rescue
- R15, R17, R19, R22, R23, R26, R27, R30, R31: symbol TFG20:R309 -> TFG20-rescue:R309-TFG20-TFG20-rescue
- R16, R18, R20, R24, R25, R28, R29, R32, R33: symbol TFG20:R619 -> TFG20-rescue:R619-TFG20-TFG20-rescue
Changed lines of the file:
@@
 $EndComp
 $Comp
-L TFG20:ADS7924IRTER IC?
+L TFG20-rescue:ADS7924IRTER-TFG20-TFG20-rescue IC?
 U 1 1 5F235551
 P 1930 3770
@@
 $EndComp
 $Comp
-L TFG20:R100 R?
+L TFG20-rescue:R100-TFG20-TFG20-rescue R?
 U 1 1 5F23555E
 P 1830 5270
@@
 $EndComp
 $Comp
-L TFG20:R100 R?
+L TFG20-rescue:R100-TFG20-TFG20-rescue R?
 U 1 1 5F235564
 P 1730 5270
@@
 $EndComp
 $Comp
-L TFG20:R100 R?
+L TFG20-rescue:R100-TFG20-TFG20-rescue R?
 U 1 1 5F23556A
 P 1630 5270
@@
 $EndComp
 $Comp
-L TFG20:R10k R?
+L TFG20-rescue:R10k-TFG20-TFG20-rescue R?
 U 1 1 5F235574
 P 1380 3070
@@
 $EndComp
 $Comp
-L TFG20:R10k R?
+L TFG20-rescue:R10k-TFG20-TFG20-rescue R?
 U 1 1 5F23557A
 P 1380 3270
@@
 $EndComp
 $Comp
-L TFG20:C100n C?
+L TFG20-rescue:C100n-TFG20-TFG20-rescue C?
 U 1 1 5F235588
 P 5070 3970
@@
 $EndComp
 $Comp
-L TFG20:C10u C?
+L TFG20-rescue:C10u-TFG20-TFG20-rescue C?
 U 1 1 5F23558E
 P 3280 4520
@@
 $EndComp
 $Comp
-L TFG20:C100n C?
+L TFG20-rescue:C100n-TFG20-TFG20-rescue C?
 U 1 1 5F235597
 P 2930 4620
@@
 $EndComp
 $Comp
-L TFG20:BLM18KG331SN1D FB?
+L TFG20-rescue:BLM18KG331SN1D-TFG20-TFG20-rescue FB?
 U 1 1 5F2355A6
 P 5450 3820
@@
 $EndComp
 $Comp
-L TFG20:BLM18KG331SN1D FB?
+L TFG20-rescue:BLM18KG331SN1D-TFG20-TFG20-rescue FB?
 U 1 1 5F2355B2
 P 3130 3960
@@
 $EndComp
 $Comp
-L TFG20:C100n C?
+L TFG20-rescue:C100n-TFG20-TFG20-rescue C?
 U 1 1 5F2355B8
 P 2480 3270
@@
 $EndComp
 $Comp
-L TFG20:NCP114BSN330T1G IC?
+L TFG20-rescue:NCP114BSN330T1G-TFG20-TFG20-rescue IC?
 U 1 1 5F2355C5
 P 4320 4270
@@
 $EndComp
 $Comp
-L TFG20:R100 R35
+L TFG20-rescue:R100-TFG20-TFG20-rescue R35
 U 1 1 5F2CC32F
 P 10770 4840
@@
 $EndComp
 $Comp
-L TFG20:R100 R?
+L TFG20-rescue:R100-TFG20-TFG20-rescue R?
 U 1 1 5F235558
 P 1930 5270
@@
 $EndComp
 $Comp
-L TFG20:R619 R24
+L TFG20-rescue:R619-TFG20-TFG20-rescue R24
 U 1 1 5F2D69E5
 P 9520 2340
@@
 $EndComp
 $Comp
-L TFG20:R619 R28
+L TFG20-rescue:R619-TFG20-TFG20-rescue R28
 U 1 1 5F2D74A1
 P 10020 2340
@@
 $EndComp
 $Comp
-L TFG20:R619 R32
+L TFG20-rescue:R619-TFG20-TFG20-rescue R32
 U 1 1 5F2D795E
 P 10520 2340
@@
 $EndComp
 $Comp
-L TFG20:R619 R33
+L TFG20-rescue:R619-TFG20-TFG20-rescue R33
 U 1 1 5F2D802C
 P 10520 4140
@@
 $EndComp
 $Comp
-L TFG20:R619 R29
+L TFG20-rescue:R619-TFG20-TFG20-rescue R29
 U 1 1 5F2D88F5
 P 10020 4140
@@
 $EndComp
 $Comp
-L TFG20:R619 R25
+L TFG20-rescue:R619-TFG20-TFG20-rescue R25
 U 1 1 5F2D8EEA
 P 9520 4140
@@
 $EndComp
 $Comp
-L TFG20:R619 R20
+L TFG20-rescue:R619-TFG20-TFG20-rescue R20
 U 1 1 5F2D94E4
 P 8430 4050
@@
 $EndComp
 $Comp
-L TFG20:R619 R18
+L TFG20-rescue:R619-TFG20-TFG20-rescue R18
 U 1 1 5F2D9AD4
 P 7930 4050
@@
 $EndComp
 $Comp
-L TFG20:R619 R16
+L TFG20-rescue:R619-TFG20-TFG20-rescue R16
 U 1 1 5F2DA010
 P 7430 4050
@@
 $EndComp
 $Comp
-L TFG20:R309 R15
+L TFG20-rescue:R309-TFG20-TFG20-rescue R15
 U 1 1 5F2DF09D
 P 7180 4500
@@
 $EndComp
 $Comp
-L TFG20:R309 R17
+L TFG20-rescue:R309-TFG20-TFG20-rescue R17
 U 1 1 5F2E087C
 P 7680 4500
@@
 $EndComp
 $Comp
-L TFG20:R309 R19
+L TFG20-rescue:R309-TFG20-TFG20-rescue R19
 U 1 1 5F2E0E69
 P 8180 4500
@@
 $EndComp
 $Comp
-L TFG20:R309 R23
+L TFG20-rescue:R309-TFG20-TFG20-rescue R23
 U 1 1 5F2E3179
 P 9270 4590
@@
 $EndComp
 $Comp
-L TFG20:R309 R27
+L TFG20-rescue:R309-TFG20-TFG20-rescue R27
 U 1 1 5F2E391A
 P 9770 4590
@@
 $EndComp
 $Comp
-L TFG20:R309 R31
+L TFG20-rescue:R309-TFG20-TFG20-rescue R31
 U 1 1 5F2E4D51
 P 10270 4590
@@
 $EndComp
 $Comp
-L TFG20:R309 R22
+L TFG20-rescue:R309-TFG20-TFG20-rescue R22
 U 1 1 5F2E5729
 P 9270 2790
@@
 $EndComp
 $Comp
-L TFG20:R309 R26
+L TFG20-rescue:R309-TFG20-TFG20-rescue R26
 U 1 1 5F2E6340
 P 9770 2790
@@
 $EndComp
 $Comp
-L TFG20:R309 R30
+L TFG20-rescue:R309-TFG20-TFG20-rescue R30
 U 1 1 5F2E6B81
 P 10270 2790
@@
 $EndComp
 $Comp
-L TFG20:R100 R21
+L TFG20-rescue:R100-TFG20-TFG20-rescue R21
 U 1 1 5F2E84D9
 P 8680 4750
@@
 $EndComp
 $Comp
-L TFG20:R100 R34
+L TFG20-rescue:R100-TFG20-TFG20-rescue R34
 U 1 1 5F2E8F1E
 P 10770 3040
@@
 AREF
 $Comp
-L TFG20:L77HDE15SD1CH4RHNVGA J5
+L TFG20-rescue:L77HDE15SD1CH4RHNVGA-TFG20-TFG20-rescue J5
 U 1 1 5F38DEC7
 P 7520 1770
