File: KiCad project/ICE40.sch (KiCad schematic (older format))
At the start: 36 parts, among them IC3 iCE40HX4K-TQ144, IC4 W25Q32JVSSIQ

Commit message: Update
Parts:
- C10: renamed from C8; symbol TFG20:C100n -> TFG20-rescue:C100n-TFG20-TFG20-rescue
- C11: renamed from C10; symbol TFG20:C100n -> TFG20-rescue:C100n-TFG20-TFG20-rescue
- C12: renamed from C20; symbol TFG20:C100n -> TFG20-rescue:C100n-TFG20-TFG20-rescue
- C13: renamed from C14; symbol TFG20:C100n -> TFG20-rescue:C100n-TFG20-TFG20-rescue
- C14: renamed from C11; symbol TFG20:C100n -> TFG20-rescue:C100n-TFG20-TFG20-rescue
- C15: renamed from C21; symbol TFG20:C100n -> TFG20-rescue:C100n-TFG20-TFG20-rescue
- C16: symbol TFG20:C10u -> TFG20-rescue:C10u-TFG20-TFG20-rescue
- C17: renamed from C13; symbol TFG20:C100n -> TFG20-rescue:C100n-TFG20-TFG20-rescue
- C18: renamed from C22; symbol TFG20:C100n -> TFG20-rescue:C100n-TFG20-TFG20-rescue
- C19: renamed from C15; symbol TFG20:C100n -> TFG20-rescue:C100n-TFG20-TFG20-rescue
- C20: renamed from C23; symbol TFG20:C100n -> TFG20-rescue:C100n-TFG20-TFG20-rescue
- C21: renamed from C17; symbol TFG20:C100n -> TFG20-rescue:C100n-TFG20-TFG20-rescue
- C22: renamed from C18; symbol TFG20:C100n -> TFG20-rescue:C100n-TFG20-TFG20-rescue
- C23: renamed from C19; symbol TFG20:C100n -> TFG20-rescue:C100n-TFG20-TFG20-rescue
- C24: symbol TFG20:C100n -> TFG20-rescue:C100n-TFG20-TFG20-rescue
- C7: renamed from C9; symbol TFG20:C100n -> TFG20-rescue:C100n-TFG20-TFG20-rescue
- C8: renamed from C7; symbol TFG20:C100n -> TFG20-rescue:C100n-TFG20-TFG20-rescue
- C9: renamed from C12; symbol TFG20:C10u -> TFG20-rescue:C10u-TFG20-TFG20-rescue
- D2: symbol TFG20:D_Schottky -> TFG20-rescue:D_Schottky-TFG20-TFG20-rescue
- IC3: symbol TFG20:iCE40HX4K-TQ144 -> TFG20-rescue:iCE40HX4K-TQ144-TFG20-TFG20-rescue
- IC4: symbol TFG20:W25Q32JVSSIQ -> TFG20-rescue:W25Q32JVSSIQ-TFG20-TFG20-rescue
- LED_FP1: symbol TFG20:LED_AMARILLO -> TFG20-rescue:LED_AMARILLO-TFG20-TFG20-rescue
- R36, R44, R45, R46, R47, R48: symbol TFG20:R10k -> TFG20-rescue:R10k-TFG20-TFG20-rescue
- R37: symbol TFG20:R2k2 -> TFG20-rescue:R2k2-TFG20-TFG20-rescue
- R38: renamed from R40; symbol TFG20:R100 -> TFG20-rescue:R100-TFG20-TFG20-rescue
- R39: renamed from R38; symbol TFG20:R470 -> TFG20-rescue:R470-TFG20-TFG20-rescue
- R40: renamed from R39; symbol TFG20:R470 -> TFG20-rescue:R470-TFG20-TFG20-rescue
- R41: symbol TFG20:R470 -> TFG20-rescue:R470-TFG20-TFG20-rescue
- R42: renamed from R43; symbol TFG20:R100 -> TFG20-rescue:R100-TFG20-TFG20-rescue
- R43: renamed from R42; symbol TFG20:R470 -> TFG20-rescue:R470-TFG20-TFG20-rescue
- R49: symbol TFG20:R1K -> TFG20-rescue:R1K-TFG20-TFG20-rescue
Connections:
- net U_SW1: now also IC3.38 (IOB_57); no longer IC3.37 (IOB_56)
- net U_SW2: now also IC3.37 (IOB_56); no longer IC3.38 (IOB_57)
- net LED0 renamed LED_1
- net LED1 renamed LED_2
- net LED2 renamed LED_0
- net LED3 renamed LED_3
Other:
- moved on the sheet: C12, C13, C15, C16, C18, C20, C23, C7, C9, D2, R38, R42
