File: KiCad project/IO.sch (KiCad schematic (older format))
At the start: 22 parts, among them J1 10129381-908002BLF, J2 10129381-908002BLF, J3 10129381-908002BLF, J4 10129381-908002BLF

Commit message: Update
Parts:
- C1, C2: symbol TFG20:C100n -> TFG20-rescue:C100n-TFG20-TFG20-rescue
- D1: symbol TFG20:D_Schottky -> TFG20-rescue:D_Schottky-TFG20-TFG20-rescue
- FPGA_R1, USW1, USW2: symbol TFG20:FSM2JLH -> TFG20-rescue:FSM2JLH-TFG20-TFG20-rescue
- J1: renamed from J4; symbol TFG20:10129381-908002BLF -> TFG20-rescue:10129381-908002BLF-TFG20-TFG20-rescue
- J2: renamed from J3; symbol TFG20:10129381-908002BLF -> TFG20-rescue:10129381-908002BLF-TFG20-TFG20-rescue
- J3: renamed from J1; symbol TFG20:10129381-908002BLF -> TFG20-rescue:10129381-908002BLF-TFG20-TFG20-rescue
- J4: renamed from J2; symbol TFG20:10129381-908002BLF -> TFG20-rescue:10129381-908002BLF-TFG20-TFG20-rescue
- LED_1: renamed from LED1; symbol TFG20:LED_AMARILLO -> TFG20-rescue:LED_AMARILLO-TFG20-TFG20-rescue
- LED_2: renamed from LED2; symbol TFG20:LED_AZUL -> TFG20-rescue:LED_AZUL-TFG20-TFG20-rescue
- LED_3: renamed from LED3; symbol TFG20:LED_VERDE -> TFG20-rescue:LED_VERDE-TFG20-TFG20-rescue
- LED_4: renamed from LED4; symbol TFG20:LED_ROJO -> TFG20-rescue:LED_ROJO-TFG20-TFG20-rescue
- R1: symbol TFG20:R10k -> TFG20-rescue:R10k-TFG20-TFG20-rescue
- R2: renamed from R5; symbol TFG20:R470 -> TFG20-rescue:R470-TFG20-TFG20-rescue
- R3: renamed from R6; symbol TFG20:R470 -> TFG20-rescue:R470-TFG20-TFG20-rescue
- R4: renamed from R7; symbol TFG20:R470 -> TFG20-rescue:R470-TFG20-TFG20-rescue
- R5: renamed from R8; symbol TFG20:R470 -> TFG20-rescue:R470-TFG20-TFG20-rescue
- R6: renamed from R2; symbol TFG20:R10k -> TFG20-rescue:R10k-TFG20-TFG20-rescue
- R7: renamed from R3; symbol TFG20:R1K -> TFG20-rescue:R1K-TFG20-TFG20-rescue
- R8: renamed from R4; symbol TFG20:R10k -> TFG20-rescue:R10k-TFG20-TFG20-rescue
Connections:
- net U_SW1: now also C2.1, R6.1, USW2.3 (NO_1), USW2.4 (NO_2); no longer C1.1, R1.1, USW1.3 (NO_1), USW1.4 (NO_2)
- net U_SW2: now also C1.1, R1.1, USW1.3 (NO_1), USW1.4 (NO_2); no longer C2.1, R6.1, USW2.3 (NO_1), USW2.4 (NO_2)
- net LED0 renamed LED_1
- net LED1 renamed LED_2
- net LED2 renamed LED_0
- net LED3 renamed LED_3
Other:
- moved on the sheet: C1, C2, D1, FPGA_R1, J1, J2, J3, J4, LED_1, LED_2, LED_3, LED_4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
