File: KiCad project/SRAM.sch (KiCad schematic (older format))
At the start: 12 parts, among them IC6 IS61WV25616EDBLL-10TLI, U3 SN74ALVCH162827

Commit message: Update
Parts:
- C53, C54, C55, C56, C57, C58: symbol TFG20:C100n -> TFG20-rescue:C100n-TFG20-TFG20-rescue
- IC6: symbol TFG20:IS61WV25616EDBLL-10TLI -> TFG20-rescue:IS61WV25616EDBLL-10TLI-TFG20-TFG20-rescue
- R69, R70, R71, R72: symbol TFG20:R10k -> TFG20-rescue:R10k-TFG20-TFG20-rescue
- U3: symbol TFG20:SN74ALVCH162827 -> TFG20-rescue:SN74ALVCH162827-TFG20-TFG20-rescue
Other:
- moved on the sheet: C53, C54, C55, C56, R69, R70, R71, R72, U3
