File: KiCad project/TFG20.kicad_pcb (KiCad board)
At the start: 4 copper layers, 117.6 x 86.9 mm, 216 parts, among them IC1 ADS7924IRTER, IC2 NCP114BSN330T1G, IC3 iCE40HX4K-TQ144, IC4 W25Q32JVSSIQ, IC5 NCP708MU330TAG, IC6 IS61WV25616EDBLL-10TLI, IC7 93LC56C-I_SN, J1 10129381-908002BLF, J10 Micro_SD_Card, J11 USB_C_Receptacle_USB2.0, J12 10129381-908002BLF, J13 10129381-908002BLF, J14 10129381-908002BLF, J15 10129381-908002BLF, J16 10129378-902001BLF, J17 10129378-902001BLF, J2 10129381-908002BLF, J3 10129381-908002BLF, J4 10129381-908002BLF, J5 L77HDE15SD1CH4RHNVGA, J6 10129381-908002BLF, J7 10129381-908002BLF, J8 1761681-3, J9 10129381-908002BLF, Q1 DMP1005UFDF-7, U1 STM32F091VCTx, U2 PAM2306AYPKB, U3 SN74ALVCH162827, U4 FT2232H, Y1 ECS-320-12-33B-7KM-TR

Commit message: Update
Parts:
- removed D5: LED_AZUL, Diode_SMD:D_0402_1005Metric
- added J10: Conn_01x01, Connector_PinHeader_2.54mm:PinHeader_1x01_P2.54mm_Vertical, F.Cu at (60.3, 50.5)
- added J13: 10129381-908002BLF, TFG_20:HDRV8W67P254_2X4_1016X483X858P, F.Cu at (20.1, 121.6)
- added J18: 10129381-908002BLF, TFG_20:HDRV8W67P254_2X4_1016X483X858P, F.Cu at (20.0, 40.7)
- added LED2: LED_AZUL, LED_SMD:LED_0603_1608Metric, F.Cu at (128.9, 87.9)
- C46, C48: value 10u -> C10u; footprint TFG_20:CAPC2012X135N -> Capacitor_SMD:C_0603_1608Metric
- C51, C52: value 10u -> C10u; footprint TFG_20:CAPC1608X90N -> Capacitor_SMD:C_0603_1608Metric
- R61, R62: footprint Resistor_SMD:R_0805_2012Metric -> Resistor_SMD:R_0402_1005Metric
- moved C52 11.1 mm to (46.6, 120.2), turned to 0 degrees
- moved C48 5.98 mm to (34.6, 111.9)
- moved C46 5.88 mm to (34.6, 117.9)
- moved J11 4.79 mm to (32.7, 44.1)
- moved C51 4.61 mm to (39.1, 109.9)
- moved C34 3.74 mm to (33.4, 53.0), turned to 180 degrees
- moved C27 1.90 mm to (62.0, 69.8), turned to 180 degrees
- moved R62 0.45 mm to (121.1, 99.5)
- moved C36 0.27 mm to (37.0, 52.9)
- moved R61 0.26 mm to (126.5, 100.9)
- renumbered C8 to C10, C10 to C11, C20 to C12, C14 to C13, C11 to C14, C21 to C15, C13 to C17, C22 to C18, C15 to C19, C23 to C20, C17 to C21, C18 to C22, C19 to C23, C9 to C7, C7 to C8, C12 to C9, J4 to J1, J10 to J11, J11 to J12, J12 to J14, J13 to J15, J14 to J16, J15 to J17, J16 to J19, J3 to J2, J17 to J20, J1 to J3, J2 to J4, LED9 to LED1, LED1 to LED_1, LED2 to LED_2, LED3 to LED_3, LED4 to LED_4, LED5 to LED_5, LED6 to LED_6, LED7 to LED_7, LED8 to LED_8, R5 to R2, R6 to R3, R40 to R38, R38 to R39, R7 to R4, R39 to R40, R43 to R42, R42 to R43, R8 to R5, R2 to R6, R3 to R7, R4 to R8
Connections:
- net LED0 renamed LED_1
- net LED1 renamed LED_2
- net LED2 renamed LED_0
- net LED3 renamed LED_3
- net LED4 renamed LED_6
- net LED5 renamed LED_7
- net LED6 renamed LED_4
- net LED7 renamed LED_5
- C1 pad 1: U_SW1 -> U_SW2
- C2 pad 1: U_SW2 -> U_SW1
- IC3 pad 37: U_SW1 -> U_SW2
- IC3 pad 38: U_SW2 -> U_SW1
- R1 pad 1: U_SW1 -> U_SW2
- R6 pad 1: U_SW2 -> U_SW1
- USW1 pad 3: U_SW1 -> U_SW2
- USW1 pad 4: U_SW1 -> U_SW2
- USW2 pad 3: U_SW2 -> U_SW1
- USW2 pad 4: U_SW2 -> U_SW1
Routing:
- net /uC/SD_D0: track 76.8 -> 66.2 mm
- net /uC/SD_DI: track 72.4 -> 64.0 mm
- net +3V3: track 173.9 -> 165.6 mm
- net /uC/SD_CS: track 70.3 -> 63.1 mm
- net /uC/SD_CLK: track 76.2 -> 69.9 mm
- net U_SW2: track 58.0 -> 52.6 mm
- net U_SW1: track 52.6 -> 58.0 mm
- net GND: track 310.5 -> 313.6 mm, vias 160 -> 159
- net USB_N: track 25.9 -> 23.7 mm
- net LED_7: track 21.5 -> 23.7 mm
- net /uC/VDDA: track 9.80 -> 11.5 mm
- net LED_6: track 20.8 -> 22.4 mm
- net LED_4: track 21.9 -> 23.6 mm
- net LED_5: track 21.3 -> 23.0 mm
- net /uC/NRST: track 67.3 -> 69.0 mm
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Other:
- board text added: "3V3"
- board text added: "5V"
- board text added: "LED_P_FPGA"
- board text added: "LED_P_uC"
- board text added: "NRST"
- board text added: "PROG"
- board text added: "SW1"
- board text added: "SW2"
- board text added: "SW3"
- board text added: "SW4"
- board text added: "|GND"
- board text removed: "LED_FP"
