File: KiCad project/USB.sch (KiCad schematic (older format))
At the start: 31 parts, among them IC7 93LC56C-I_SN, J16 10129378-902001BLF, J17 10129378-902001BLF, U4 FT2232H

Commit message: Update
Parts:
- C59, C60, C61, C62, C63, C64, C66, C67, C68, C69, C70, C71, C72, C73: symbol TFG20:C100n -> TFG20-rescue:C100n-TFG20-TFG20-rescue
- C65: symbol TFG20:C10u -> TFG20-rescue:C10u-TFG20-TFG20-rescue
- FB5, FB6: symbol TFG20:BLM18KG331SN1D -> TFG20-rescue:BLM18KG331SN1D-TFG20-TFG20-rescue
- IC7: symbol TFG20:93LC56C-I_SN -> TFG20-rescue:93LC56C-I_SN-TFG20-TFG20-rescue
- J19: renamed from J16; symbol TFG20:10129378-902001BLF -> TFG20-rescue:10129378-902001BLF-TFG20-TFG20-rescue
- J20: renamed from J17; symbol TFG20:10129378-902001BLF -> TFG20-rescue:10129378-902001BLF-TFG20-TFG20-rescue
- LED1: renamed from LED9; symbol TFG20:LED_AMARILLO -> TFG20-rescue:LED_AMARILLO-TFG20-TFG20-rescue
- O1: symbol TFG20:DSC1001CL2 -> TFG20-rescue:DSC1001CL2-TFG20-TFG20-rescue
- R73, R75, R76, R78: symbol TFG20:R10k -> TFG20-rescue:R10k-TFG20-TFG20-rescue
- R74, R80: symbol TFG20:R100 -> TFG20-rescue:R100-TFG20-TFG20-rescue
- R77: symbol TFG20:R2k2 -> TFG20-rescue:R2k2-TFG20-TFG20-rescue
- R79: symbol TFG20:R1K -> TFG20-rescue:R1K-TFG20-TFG20-rescue
