File: KiCad project/globalpower.sch (KiCad schematic (older format))
At the start: 40 parts, among them IC5 NCP708MU330TAG, J11 USB_C_Receptacle_USB2.0, J12 10129381-908002BLF, J13 10129381-908002BLF, J14 10129381-908002BLF, J15 10129381-908002BLF, Q1 DMP1005UFDF-7, U2 PAM2306AYPKB

Commit message: Update
Parts:
- removed C46, C48: 10u, TFG_20:CAPC2012X135N, symbol TFG20:LMK212ABJ106KGHT
- removed C51, C52: 10u, TFG_20:CAPC1608X90N, symbol TFG20:GRM188R61A106KE69D
- removed D5: LED_AZUL, Diode_SMD:D_0402_1005Metric, symbol TFG20:LED_AZUL
- added C46, C48, C51, C52: C10u, Capacitor_SMD:C_0603_1608Metric, symbol TFG20:C10u
- added J13, J18: 10129381-908002BLF, TFG_20:HDRV8W67P254_2X4_1016X483X858P, symbol TFG20-rescue:10129381-908002BLF-TFG20-TFG20-rescue
- added LED2: LED_AZUL, LED_SMD:LED_0603_1608Metric, symbol TFG20:LED_AZUL
- C41, C42, C43, C45: symbol TFG20:C100n -> TFG20-rescue:C100n-TFG20-TFG20-rescue
- C44, C47: symbol TFG20:C220uElect -> TFG20-rescue:C220uElect-TFG20-TFG20-rescue
- D3: symbol TFG20:824500500 -> TFG20-rescue:824500500-TFG20-TFG20-rescue
- D4: symbol TFG20:82400152 -> TFG20-rescue:82400152-TFG20-TFG20-rescue
- FB4: symbol TFG20:BLM18KG331SN1D -> TFG20-rescue:BLM18KG331SN1D-TFG20-TFG20-rescue
- IC5: symbol TFG20:NCP708MU330TAG -> TFG20-rescue:NCP708MU330TAG-TFG20-TFG20-rescue
- J12: renamed from J11; symbol TFG20:USB_C_Receptacle_USB2.0 -> TFG20-rescue:USB_C_Receptacle_USB2.0-TFG20-TFG20-rescue
- J14: renamed from J12; symbol TFG20:10129381-908002BLF -> TFG20-rescue:10129381-908002BLF-TFG20-TFG20-rescue
- J15: renamed from J13; symbol TFG20:10129381-908002BLF -> TFG20-rescue:10129381-908002BLF-TFG20-TFG20-rescue
- J16: renamed from J14; symbol TFG20:10129381-908002BLF -> TFG20-rescue:10129381-908002BLF-TFG20-TFG20-rescue
- J17: renamed from J15; symbol TFG20:10129381-908002BLF -> TFG20-rescue:10129381-908002BLF-TFG20-TFG20-rescue
- L1, L2: symbol TFG20:LQH5BPN4R7NT0L -> TFG20-rescue:LQH5BPN4R7NT0L-TFG20-TFG20-rescue
- PWR_LED1: symbol TFG20:LED_AZUL -> TFG20-rescue:LED_AZUL-TFG20-TFG20-rescue
- Q1: symbol TFG20:DMP1005UFDF-7 -> TFG20-rescue:DMP1005UFDF-7-TFG20-TFG20-rescue
- R58: symbol TFG20:R100 -> TFG20-rescue:R100-TFG20-TFG20-rescue
- R59, R60: symbol TFG20:R10k -> TFG20-rescue:R10k-TFG20-TFG20-rescue
- R61, R62: footprint Resistor_SMD:R_0805_2012Metric -> Resistor_SMD:R_0402_1005Metric
- R63, R65: symbol TFG20:R2k2 -> TFG20-rescue:R2k2-TFG20-TFG20-rescue
- S1: symbol TFG20:PCM12SMTR -> TFG20-rescue:PCM12SMTR-TFG20-TFG20-rescue
- Z1: symbol TFG20:1SMB5913BT3G -> TFG20-rescue:1SMB5913BT3G-TFG20-TFG20-rescue
Connections:
- net +1V2: now also C52.1
- net +3V3: now also C51.1, J18.1, J18.3, J18.5, J18.7
- net +5F: now also C46.1, C48.1
- net +5V: now also J13.1, J13.3, J13.5, J13.7
- net GND: now also C46.2, C48.2, C51.2, C52.2, J13.2, J13.4, J13.6, J13.8, J18.2, J18.4, J18.6, J18.8, LED2.1 (K)
- net at R65.2: now also LED2.2 (A)
Other:
- moved on the sheet: J14, J15, J16, J17
