File: KiCad project/uC.sch (KiCad schematic (older format))
At the start: 39 parts, among them J10 Micro_SD_Card, J6 10129381-908002BLF, J7 10129381-908002BLF, J8 1761681-3, J9 10129381-908002BLF, U1 STM32F091VCTx, Y1 ECS-320-12-33B-7KM-TR

Commit message: Update
Parts:
- added J10: Conn_01x01, Connector_PinHeader_2.54mm:PinHeader_1x01_P2.54mm_Vertical, symbol Connector_Generic:Conn_01x01
- C25, C33: symbol TFG20:C4.7uElect -> TFG20-rescue:C4.7uElect-TFG20-TFG20-rescue
- C26: symbol TFG20:C1u -> TFG20-rescue:C1u-TFG20-TFG20-rescue
- C27: symbol TFG20:C10n -> TFG20-rescue:C10n-TFG20-TFG20-rescue
- C28, C29, C30, C31, C32, C35, C36, C37, C40: symbol TFG20:C100n -> TFG20-rescue:C100n-TFG20-TFG20-rescue
- C34: symbol TFG20:C10u -> TFG20-rescue:C10u-TFG20-TFG20-rescue
- C38, C39: symbol TFG20:C20p -> TFG20-rescue:C20p-TFG20-TFG20-rescue
- FB3: symbol TFG20:BLM18KG331SN1D -> TFG20-rescue:BLM18KG331SN1D-TFG20-TFG20-rescue
- J11: renamed from J10; symbol TFG20:Micro_SD_Card -> TFG20-rescue:Micro_SD_Card-TFG20-TFG20-rescue
- J6, J7, J9: symbol TFG20:10129381-908002BLF -> TFG20-rescue:10129381-908002BLF-TFG20-TFG20-rescue
- J8: symbol TFG20:1761681-3 -> TFG20-rescue:1761681-3-TFG20-TFG20-rescue
- LED_5: renamed from LED5; symbol TFG20:LED_ROJO -> TFG20-rescue:LED_ROJO-TFG20-TFG20-rescue
- LED_6: renamed from LED6; symbol TFG20:LED_VERDE -> TFG20-rescue:LED_VERDE-TFG20-TFG20-rescue
- LED_7: renamed from LED7; symbol TFG20:LED_AZUL -> TFG20-rescue:LED_AZUL-TFG20-TFG20-rescue
- LED_8: renamed from LED8; symbol TFG20:LED_AMARILLO -> TFG20-rescue:LED_AMARILLO-TFG20-TFG20-rescue
- R50, R51, R52, R53: symbol TFG20:R470 -> TFG20-rescue:R470-TFG20-TFG20-rescue
- R54, R55, R57: symbol TFG20:R10k -> TFG20-rescue:R10k-TFG20-TFG20-rescue
- R56: symbol TFG20:R1K -> TFG20-rescue:R1K-TFG20-TFG20-rescue
- U1: symbol TFG20:STM32F091VCTx -> TFG20-rescue:STM32F091VCTx-TFG20-TFG20-rescue
- USW3, USW4, uC_R1: symbol TFG20:FSM2JLH -> TFG20-rescue:FSM2JLH-TFG20-TFG20-rescue
- Y1: symbol TFG20:ECS-320-12-33B-7KM-TR -> TFG20-rescue:ECS-320-12-33B-7KM-TR-TFG20-TFG20-rescue
Connections:
- net NRST: now also J10.1 (Pin_1)
- net LED4 renamed LED_6
- net LED5 renamed LED_7
- net LED6 renamed LED_4
- net LED7 renamed LED_5
